Commit message: Inverse Kinematics work

File: parametric_hexapod.urdf (robot description, URDF)
Before this commit: robot pexod, 19 links, 18 joints
Links:
- link leg_1_3: geometry collision box size=eval[2*{r3}] eval[2*{r3}] eval[{l3}-{r3}]; collision sphere radius={r3}
- link leg_2_3: geometry collision box size=eval[2*{r3}] eval[2*{r3}] eval[{l3}-{r3}]; collision sphere radius={r3}
- link leg_3_3: geometry collision box size=eval[2*{r3}] eval[2*{r3}] eval[{l3}-{r3}]; collision sphere radius={r3}
- link leg_4_3: geometry collision box size=eval[2*{r3}] eval[2*{r3}] eval[{l3}-{r3}]; collision sphere radius={r3}
- link leg_5_3: geometry collision box size=eval[2*{r3}] eval[2*{r3}] eval[{l3}-{r3}]; collision sphere radius={r3}
Joints:
- joint leg_0_1_2: axis 1 0 0 -> -1 0 0
- joint leg_0_2_3: origin xyz=0 {l2} 0 rpy=-1.57079632679 0 0 -> xyz=0 {l2} 0 rpy=0 0 0
- joint leg_1_1_2: axis 1 0 0 -> -1 0 0
- joint leg_1_2_3: origin xyz=0 {l2} 0 rpy=-1.57079632679 0 0 -> xyz=0 {l2} 0 rpy=0 0 0
- joint leg_2_1_2: axis 1 0 0 -> -1 0 0
- joint leg_2_2_3: origin xyz=0 {l2} 0 rpy=-1.57079632679 0 0 -> xyz=0 {l2} 0 rpy=0 0 0
- joint leg_3_1_2: axis -1 0 0 -> 1 0 0
- joint leg_3_2_3: origin xyz=0 -{l2} 0 rpy=1.57079632679 0 0 -> xyz=0 -{l2} 0 rpy=0 0 0
- joint leg_4_1_2: axis -1 0 0 -> 1 0 0
- joint leg_4_2_3: origin xyz=0 -{l2} 0 rpy=1.57079632679 0 0 -> xyz=0 -{l2} 0 rpy=0 0 0
- joint leg_5_1_2: axis -1 0 0 -> 1 0 0
- joint leg_5_2_3: origin xyz=0 -{l2} 0 rpy=1.57079632679 0 0 -> xyz=0 -{l2} 0 rpy=0 0 0

Commit message: Basic Walker implemented. There is an issue with the body height

File: parametric_hexapod.urdf (robot description, URDF)
Before this commit: robot pexod, 19 links, 18 joints
Links:
- link leg_0_3: geometry collision box size=eval[2*{r3}] eval[2*{r3}] eval[{l3}-{r3}]; collision sphere radius={r3}

Commit message: fixed height of robot

File: parametric_hexapod.urdf (robot description, URDF)
Before this commit: robot pexod, 19 links, 18 joints
Links:
- link leg_0_1: geometry collision box size=eval[2*{r1}] eval[2*{r1}] {l1}; visual cylinder length={l1} radius={r1}
- link leg_0_2: geometry collision box size=eval[2*{r2}] eval[2*{r2}] {l2}; visual cylinder length={l2} radius={r2}
- link leg_0_3: geometry collision box size=eval[2*{r3}] eval[2*{r3}] eval[{l3}-{r3}]; collision sphere radius={r3}
- link leg_1_1: geometry collision box size=eval[2*{r1}] eval[2*{r1}] {l1}; visual cylinder length={l1} radius={r1}
- link leg_1_2: geometry collision box size=eval[2*{r2}] eval[2*{r2}] {l2}; visual cylinder length={l2} radius={r2}
- link leg_2_1: geometry collision box size=eval[2*{r1}] eval[2*{r1}] {l1}; visual cylinder length={l1} radius={r1}
- link leg_2_2: geometry collision box size=eval[2*{r2}] eval[2*{r2}] {l2}; visual cylinder length={l2} radius={r2}
- link leg_3_1: geometry collision box size=eval[2*{r1}] eval[2*{r1}] {l1}; visual cylinder length={l1} radius={r1}
- link leg_3_2: geometry collision box size=eval[2*{r2}] eval[2*{r2}] {l2}; visual cylinder length={l2} radius={r2}
- link leg_4_1: geometry collision box size=eval[2*{r1}] eval[2*{r1}] {l1}; visual cylinder length={l1} radius={r1}
- link leg_4_2: geometry collision box size=eval[2*{r2}] eval[2*{r2}] {l2}; visual cylinder length={l2} radius={r2}
- link leg_5_1: geometry collision box size=eval[2*{r1}] eval[2*{r1}] {l1}; visual cylinder length={l1} radius={r1}
- link leg_5_2: geometry collision box size=eval[2*{r2}] eval[2*{r2}] {l2}; visual cylinder length={l2} radius={r2}
